Commit message: add ekf from robot localization

File: src/description/rover_description.urdf (robot description, URDF)
Before this commit: robot rover, 2 links, 1 joints
Links:
- added link laser
Joints:
- added joint base_link_to_laser: type fixed, parent base_link, child laser, origin xyz=0.2 0.0 0.1 rpy=0 0 0

Commit message: ros2_control urdf

File: src/description/rover_description.urdf (robot description, URDF)
Before this commit: robot rover, 3 links, 2 joints
Links:
- added link camera_link
Joints:
- added joint base_link_to_camera_link: type fixed, parent base_link, child camera_link, origin xyz=0.2 0.0 0.1 rpy=0 0 0

Commit message: camera IMU optical

File: src/description/rover_description.urdf (robot description, URDF)
Before this commit: robot rover, 4 links, 3 joints
Links:
- added link camera_imu_frame
- added link camera_imu_optical_frame
Joints:
- added joint camera_imu_to_camera_imu_optical: type fixed, parent camera_imu_frame, child camera_imu_optical_frame, origin xyz=0 0 0 rpy=${-pi/2} 0 ${-pi/2}
- added joint camera_link_to_camera_imu_frame: type fixed, parent camera_link, child camera_imu_frame, origin xyz=0 0 0 rpy=${pi} 0 0

Commit message: clean up rover description package

File: src/description/rover_description.urdf (robot description, URDF)
Before this commit: robot rover, 6 links, 5 joints
Joints:
- joint camera_imu_to_camera_imu_optical: origin xyz=0 0 0 rpy=${-pi/2} 0 ${-pi/2} -> xyz=0 0 0 rpy=-1.5707963 0 -1.5707963
- joint camera_link_to_camera_imu_frame: origin xyz=0 0 0 rpy=${pi} 0 0 -> xyz=0 0 0 rpy=0 0 0
